Commit message: modify urdf

File: limo_sim/urdf/limo.gazebo.xacro (robot description, xacro)
@@ -26,3 +26,24 @@
         <material>Gazebo/FlatBlack</material>
     </gazebo>
+    <gazebo reference="wheel_rear_left_link">
+        <mu1>0.1</mu1>
+        <mu2>0.1</mu2>
+        <kp>500000.0</kp>
+        <kd>10.0</kd>
+        <minDepth>0.001</minDepth>
+        <maxVel>0.1</maxVel>
+        <fdir1>1 0 0</fdir1>
+        <material>Gazebo/FlatBlack</material>
+    </gazebo>
+    <gazebo reference="imu_link">
+        <sensor type="imu" name="imu">
+            <always_on>true</always_on>
+            <visualize>$(arg imu_visual)</visualize>
+        </sensor>
+        <material>Gazebo/FlatBlack</material>
+    </gazebo>
+    <gazebo>
+        <plugin name="limo_diff_controller" filename="libgazebo_ros_diff_drive.so">
+        </plugin>
+    </gazebo>
 </robot>

File: limo_sim/urdf/limo.urdf.xacro (robot description, xacro)
@@ -65,4 +65,52 @@
   </join>
   <link name="wheel_rear_left_link">
+    <visual>
+      <origin xyz="0 0 0" rpy="1.57 0 0"/>
+      <geometry>
+        <mesh filename="package://limo_sim/meshes/rear_left_tire.stl" scale="1 1 1"/>
+      </geometry>
+      <material name="dark"/>
+    </visual>
+    <collision>
+      <origin xyz="0 0 0" rpy="0 0 0"/>
+      <geometry>
+        <cylinder length="0.018" radius="0.033" />
+      </geometry>
+    </collision>
+    <inertial>
+      <origin xyz="0 0 0"/>
+      <mass value="2.8498940e-02" />
+      <inertia ixx="1.1175580e-05" ixy="-4.2369783e-11" ixz="-5.9381719e-09"
+               iyy="1.1192413e-05" iyz="-1.4400107e-11"
+               izz="2.0712558e-05" />
+    </inertial>
+  </link>
+  <join name="wheel_rear_right_joint" type="continuous">
+    <parent link="base_link" />
+    <child link="wheel_rear_right_link"/>
+    <origin xyz="0.0 -0.08 0.023" rpy="-1.57 0 0" />
+    <axis xyz="0 0 1" />
+  </join>
+  <link name="wheel_rear_right_link">
+    <visual>
+      <origin xyz="0 0 0" rpy="1.57 0 0" />
+      <geometry>
+        <mesh filename="package://limo_sim/meshes/rear_right_tire.stl" scale="1 1 1"/>
+      </geometry>
+      <material name="dark"/>
+    </visual>
+    <collision>
+      <origin xyz="0 0 0" rpy="0 0 0"/>
+      <geometry>
+        <cylinder length="0.018" radius="0.033"/>
+      </geometry>
+    </collision>
+    <inertial>
+      <origin xyz="0 0 0"/>
+      <mass value="2.8498940e-02" />
+      <inertia ixx="1.1175580e-05" ixy="-4.2369783e-11" ixz="-5.9381719e-09"
+               iyy="1.1192413e-05" iyz="-1.4400107e-11"
+               izz="2.0712558e-05" />
+    </inertial>
   </link>
   <join name="wheel_front_right_joint" type="continuous" >

Commit message: add gazebo urdf

File: limo_sim/urdf/limo.gazebo.xacro (robot description, xacro)
@@ -44,6 +44,86 @@
     </gazebo>
     <gazebo>
-        <plugin name="limo_diff_controller" filename="libgazebo_ros_diff_drive.so">
+        <plugin name="limo_diff_controller" filename="liblimo_ros_4_wheel_diff_drive.so">
+            <commandTopic>cmd_vel</commandTopic>
+            <odometryTopic>odom</odometryTopic>
+            <odometryFrame>odom</odometryFrame>
+            <odometrySource>world</odometrySource>
+            <publishOdomTF>true</publishOdomTF>
+            <robotBaseFrame>base_footprint</robotBaseFrame>
+            <publishWheelTF>false</publishWheelTF>
+            <publishTf>true</publishTf>
+            <publishWheelJointState>true</publishWheelJointState>
+            <legacyMode>false</legacyMode>
+            <updateRate>30</updateRate>
+            <frontLeftJoint>wheel_front_left_joint</frontLeftJoint>
+            <frontRightJoint>wheel_front_right_joint</frontRightJoint>
+            <rearLeftJoint>wheel_rear_left_joint</rearLeftJoint>
+            <rearRightJoint>wheel_rear_right_joint</rearRightJoint>
+            <wheelSeparation>0.160</wheelSeparation>
+            <wheelDiameter>0.066</wheelDiameter>
+            <wheelAcceleration>1</wheelAcceleration>
+            <wheelTorque>10</wheelTorque>
+            <rosDebugLevel>na</rosDebugLevel>
         </plugin>
     </gazebo>
+    <gazebo>
+        <plugin name="imu_plugin" filename="libgazebo_ros_imu.so">
+            <alwaysOn>true</alwaysOn>
+            <bodyName>imu_link</bodyName>
+            <frameName>imu_link</frameName>
+            <topicName>imu</topicName>
+            <serviceName>imu_service</serviceName>
+            <gaussianNoise>0.0</gaussianNoise>
+            <updateRate>0</updateRate>
+            <imu>
+                <noise>
+                  <type>gaussian</type>
+                  <rate>
+                    <mean>0.0</mean>
+                    <stddev>2e-4</stddev>
+                    <bias_mean>0.0000075</bias_mean>
+                    <bias_stddev>0.0000008</bias_stddev>
+                  </rate>
+                  <accel>
+                    <mean>0.0</mean>
+                    <stddev>1.7e-2</stddev>
+                    <bias_mean>0.1</bias_mean>
+                    <bias_stddev>0.001</bias_stddev>
+                  </accel>
+                </noise>
+              </imu>
+        </plugin>
+    </gazebo>
+    <gazebo reference="base_scan">
+        <material>Gazebo/FlatBlack</material>
+        <sensor type="ray" name="lds_lfcd_sensor">
+          <pose>0 0 0 0 0 0</pose>
+          <visualize>$(arg laser_visual)</visualize>
+          <update_rate>5</update_rate>
+          <ray>
+            <scan>
+              <horizontal>
+                <samples>360</samples>
+                <resolution>1</resolution>
+                <min_angle>0.0</min_angle>
+                <max_angle>6.28319</max_angle>
+              </horizontal>
+            </scan>
+            <range>
+              <min>0.120</min>
+              <max>3.5</max>
+              <resolution>0.015</resolution>
+            </range>
+            <noise>
+              <type>gaussian</type>
+              <mean>0.0</mean>
+              <stddev>0.01</stddev>
+            </noise>
+          </ray>
+          <plugin name="gazebo_ros_lds_lfcd_controller" filename="libgazebo_ros_laser.so">
+            <topicName>scan</topicName>
+            <frameName>base_scan</frameName>
+          </plugin>
+        </sensor>
+      </gazebo>
 </robot>

Commit message: modify urdf

File: limo_sim/urdf/limo.gazebo.xacro (robot description, xacro)
@@ -14,7 +14,7 @@
         <maxVel>0.1</maxVel>
         <fdir1>1 0 0</fdir1>
-        <material>Gazebo/FlatBlack</material>
+        <material>Gazebo/Red</material>
     </gazebo>
-    <gazebo reference="wheel_front_right_link">
+    <gazebo reference="wheel_rear_left_link">
         <mu1>0.1</mu1>
         <mu2>0.1</mu2>
@@ -24,7 +24,17 @@
         <maxVel>0.1</maxVel>
         <fdir1>1 0 0</fdir1>
-        <material>Gazebo/FlatBlack</material>
+        <material>Gazebo/Green</material>
     </gazebo>
-    <gazebo reference="wheel_rear_left_link">
+    <gazebo reference="wheel_rear_right_link">
+        <mu1>0.1</mu1>
+        <mu2>0.1</mu2>
+        <kp>500000.0</kp>
+        <kd>10.0</kd>
+        <minDepth>0.001</minDepth>
+        <maxVel>0.1</maxVel>
+        <fdir1>1 0 0</fdir1>
+        <material>Gazebo/Blue</material>
+    </gazebo>
+    <gazebo reference="wheel_front_right_link">
         <mu1>0.1</mu1>
         <mu2>0.1</mu2>

File: limo_sim/urdf/limo.urdf.xacro (robot description, xacro)
@@ -12,5 +12,5 @@
       <origin xyz="-0.032 0 0.0" rpy="0 0 0"/>
       <geometry>
-        <mesh filename="package://limo_sim/meshes/base_link.STL" scale="1 1 1"/>
+        <mesh filename="package://limo_sim/meshes/base_link.stl" scale="1 1 1"/>
       </geometry>
       <material name="light_black"/>
@@ -30,17 +30,17 @@
     </inertial>
   </link>
-  <join name="wheel_front_left_join" type="continuous">
+  <joint name="wheel_front_left_joint" type="continuous">
     <parent link="base_link" />
     <child link="wheel_front_left_link" />
-    <origin xyz="0.11 0.11 0.023" rpy="-1.57 0 0" />
+    <origin xyz="0 0 0.023" rpy="-1.57 0 0" />
     <axis xyz="0 0 1" />
-  </join>
+  </joint>
   <link name="wheel_front_left_link">
     <visual>
       <origin xyz="0 0 0" rpy="1.57 0 0"/>
       <geometry>
-        <mesh filename="package://limo_sim/meshes/wheels/front_left_tire.stl" scale="1 1 1"/>
+        <mesh filename="package://limo_sim/meshes/wheels/front_left_tire.stl" scale="0.001 0.001 0.001"/>
       </geometry>
-      <material name="dark" />
+      <material name="red" />
     </visual>
     <collision>
@@ -58,17 +58,17 @@
       </inertial>
   </link>
-  <join name="wheel_rear_left_join" type="continuous" >
+  <joint name="wheel_rear_left_join" type="continuous" >
     <parent link="base_link" />
     <child link="wheel_rear_left_link"/>
-    <origin xyz="-0.11 0.11 0.023" rpy="-1.57 0 0" />
+    <origin xyz="0 0 0.123" rpy="-1.57 0 0" />
     <axis xyz="0 0 1" />
-  </join>
+  </joint>
   <link name="wheel_rear_left_link">
     <visual>
       <origin xyz="0 0 0" rpy="1.57 0 0"/>
       <geometry>
-        <mesh filename="package://limo_sim/meshes/rear_left_tire.stl" scale="1 1 1"/>
+        <mesh filename="package://limo_sim/meshes/wheels/rear_left_tire.stl" scale="0.001 0.001 0.001"/>
       </geometry>
-      <material name="dark"/>
+      <material name="green"/>
     </visual>
     <collision>
@@ -86,17 +86,17 @@
     </inertial>
   </link>
-  <join name="wheel_rear_right_joint" type="continuous">
+  <joint name="wheel_rear_right_joint" type="continuous">
     <parent link="base_link" />
     <child link="wheel_rear_right_link"/>
-    <origin xyz="0.0 -0.08 0.023" rpy="-1.57 0 0" />
+    <origin xyz="0 0 0.223" rpy="-1.57 0 0" />
     <axis xyz="0 0 1" />
-  </join>
+  </joint>
   <link name="wheel_rear_right_link">
     <visual>
       <origin xyz="0 0 0" rpy="1.57 0 0" />
       <geometry>
-        <mesh filename="package://limo_sim/meshes/rear_right_tire.stl" scale="1 1 1"/>
+        <mesh filename="package://limo_sim/meshes/wheels/rear_right_tire.stl" scale="0.001 0.001 0.001"/>
       </geometry>
-      <material name="dark"/>
+      <material name="blue"/>
     </visual>
     <collision>
@@ -114,15 +114,15 @@
     </inertial>
   </link>
-  <join name="wheel_front_right_joint" type="continuous" >
+  <joint name="wheel_front_right_joint" type="continuous" >
     <parent link="base_link" />
     <child link="wheel_front_right_link" />
-    <origin xyz="0.0 -0.08 0.023" rpy="-1.57 0 0"/>
+    <origin xyz="0.0 0 0.323" rpy="-1.57 0 0"/>
     <axis xyz="0 0 1"/>
-  </join>
+  </joint>
   <link name="wheel_front_right_link">
     <visual>
       <origin xyz="0 0 0" rpy="1.57 0 0" />
       <geometry>
-        <mesh filename="package://limo_sim/meshes/wheels/front_right_tire.stl" scale="1 1 1"/>
+        <mesh filename="package://limo_sim/meshes/wheels/front_right_tire.stl" scale="0.001 0.001 0.001"/>
       </geometry>
       <material name="dark"/>
@@ -157,5 +157,5 @@
       <origin xyz="0 0 0" rpy="0 0 0"/>
       <geometry>
-        <mesh filename="package://limo_sim/meshes/sensors/lds.stl" scale="1 1 1"/>
+        <mesh filename="package://limo_sim/meshes/sensors/lds.stl" scale="0.001 0.001 0.001"/>
       </geometry>
       <material name="dark" />

Commit message: limo sim , can not run

File: limo_sim/urdf/limo.gazebo.xacro (robot description, xacro)
@@ -44,5 +44,5 @@
         <maxVel>0.1</maxVel>
         <fdir1>1 0 0</fdir1>
-        <material>Gazebo/FlatBlack</material>
+        <material>Gazebo/Yellow</material>
     </gazebo>
     <gazebo reference="imu_link">
@@ -67,7 +67,7 @@
             <updateRate>30</updateRate>
             <frontLeftJoint>wheel_front_left_joint</frontLeftJoint>
-            <frontRightJoint>wheel_front_right_joint</frontRightJoint>
             <rearLeftJoint>wheel_rear_left_joint</rearLeftJoint>
             <rearRightJoint>wheel_rear_right_joint</rearRightJoint>
+            <frontRightJoint>wheel_front_right_joint</frontRightJoint>
             <wheelSeparation>0.160</wheelSeparation>
             <wheelDiameter>0.066</wheelDiameter>
@@ -136,4 +136,4 @@
           </plugin>
         </sensor>
-      </gazebo>
+    </gazebo>
 </robot>

File: limo_sim/urdf/limo.urdf.xacro (robot description, xacro)
@@ -10,5 +10,4 @@
   <link name="base_link">
     <visual>
-      <origin xyz="-0.032 0 0.0" rpy="0 0 0"/>
       <geometry>
         <mesh filename="package://limo_sim/meshes/base_link.stl" scale="1 1 1"/>
@@ -33,10 +32,9 @@
     <parent link="base_link" />
     <child link="wheel_front_left_link" />
-    <origin xyz="0 0 0.023" rpy="-1.57 0 0" />
+    <origin xyz="0.035 -0.05 0.005" rpy="0 0 -1.57" />
     <axis xyz="0 0 1" />
   </joint>
   <link name="wheel_front_left_link">
     <visual>
-      <origin xyz="0 0 0" rpy="1.57 0 0"/>
       <geometry>
         <mesh filename="package://limo_sim/meshes/wheels/front_left_tire.stl" scale="0.001 0.001 0.001"/>
@@ -58,13 +56,12 @@
       </inertial>
   </link>
-  <joint name="wheel_rear_left_join" type="continuous" >
+  <joint name="wheel_rear_left_joint" type="continuous" >
     <parent link="base_link" />
     <child link="wheel_rear_left_link"/>
-    <origin xyz="0 0 0.123" rpy="-1.57 0 0" />
+    <origin xyz="0.03 0.12 0.005" rpy="0 0 -1.57" />
     <axis xyz="0 0 1" />
   </joint>
   <link name="wheel_rear_left_link">
     <visual>
-      <origin xyz="0 0 0" rpy="1.57 0 0"/>
       <geometry>
         <mesh filename="package://limo_sim/meshes/wheels/rear_left_tire.stl" scale="0.001 0.001 0.001"/>
@@ -89,10 +86,9 @@
     <parent link="base_link" />
     <child link="wheel_rear_right_link"/>
-    <origin xyz="0 0 0.223" rpy="-1.57 0 0" />
+    <origin xyz="-0.035 0.06 0.005" rpy="0 0 1.57" />
     <axis xyz="0 0 1" />
   </joint>
   <link name="wheel_rear_right_link">
     <visual>
-      <origin xyz="0 0 0" rpy="1.57 0 0" />
       <geometry>
         <mesh filename="package://limo_sim/meshes/wheels/rear_right_tire.stl" scale="0.001 0.001 0.001"/>
@@ -117,14 +113,13 @@
     <parent link="base_link" />
     <child link="wheel_front_right_link" />
-    <origin xyz="0.0 0 0.323" rpy="-1.57 0 0"/>
+    <origin xyz="-0.035 -0.15 0.005" rpy="0 0 1.57"/>
     <axis xyz="0 0 1"/>
   </joint>
   <link name="wheel_front_right_link">
     <visual>
-      <origin xyz="0 0 0" rpy="1.57 0 0" />
       <geometry>
         <mesh filename="package://limo_sim/meshes/wheels/front_right_tire.stl" scale="0.001 0.001 0.001"/>
       </geometry>
-      <material name="dark"/>
+      <material name="yellow"/>
     </visual>
     <collision>
@@ -151,9 +146,8 @@
     <parent link="base_link"/>
     <child link="base_scan" />
-    <origin xyz="0.032 0 0.172" rpy="0 0 0"/>
+    <origin xyz="0.0 0 0.172" rpy="0 0 0"/>
   </joint>
   <link name="base_scan">
     <visual>
-      <origin xyz="0 0 0" rpy="0 0 0"/>
       <geometry>
         <mesh filename="package://limo_sim/meshes/sensors/lds.stl" scale="0.001 0.001 0.001"/>
